File: mosfetSwitch.brd (EAGLE design)
At the start: 53.3 x 82.9 mm, 29 parts, among them Q1 BC848, Q2 BC848, Q3 BC848, Q4 BC848, T1 AO4805, T2 AO4805

Commit message: BRD pridane test pady
Parts:
- added TP2, TP3, TP4, TP5: TPSB2,54, testpad:B2,54
Connections:
- net SW0: now also TP5.TP
- net SW1: now also TP4.TP
- net SW2: now also TP3.TP
- net SW3: now also TP2.TP
Routing:
- net N$8: track 15.5 -> 22.0 mm
- net N$11: track 18.5 -> 25.0 mm
- net INPUT: track 97.2 -> 100.1 mm
- net N$7: track 33.6 -> 35.1 mm
- net INPUT2: track 49.3 -> 50.4 mm
