File: mosfetSwitch.sch (EAGLE design)
At the start: 29 parts, among them Q1 BC848, Q2 BC848, Q3 BC848, Q4 BC848, T1 AO4805, T2 AO4805

Commit message: BRD pridane test pady
Parts:
- added TP2, TP3, TP4, TP5: TPSB2,54, testpad:TPSB2,54
Connections:
- net SW0: now also TP5.PP
- net SW1: now also TP4.PP
- net SW2: now also TP3.PP
- net SW3: now also TP2.PP
Changed lines of the file:
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@@
 <part name="S3" library="misc" library_urn="urn:adsk.eagle:library:4373854" deviceset="10-XX" device="3D" package3d_urn="urn:adsk.eagle:package:4373869/2"/>
 <part name="GND9" library="node_v4" deviceset="GND" device=""/>
+<part name="TP2" library="testpad" library_urn="urn:adsk.eagle:library:385" deviceset="TPS" device="B2,54" package3d_urn="urn:adsk.eagle:package:27948/1"/>
+<part name="TP3" library="testpad" library_urn="urn:adsk.eagle:library:385" deviceset="TPS" device="B2,54" package3d_urn="urn:adsk.eagle:package:27948/1"/>
+<part name="TP4" library="testpad" library_urn="urn:adsk.eagle:library:385" deviceset="TPS" device="B2,54" package3d_urn="urn:adsk.eagle:package:27948/1"/>
+<part name="TP5" library="testpad" library_urn="urn:adsk.eagle:library:385" deviceset="TPS" device="B2,54" package3d_urn="urn:adsk.eagle:package:27948/1"/>
 </parts>
 <sheets>
@@
 <instance part="GND9" gate="G$1" x="99.06" y="-20.32" smashed="yes">
 <attribute name="VALUE" x="97.536" y="-22.86" size="1.27" layer="96"/>
+</instance>
+<instance part="TP2" gate="G$1" x="66.04" y="30.48" smashed="yes">
+<attribute name="NAME" x="64.77" y="31.75" size="1.778" layer="95"/>
+<attribute name="TP_SIGNAL_NAME" x="67.31" y="29.21" size="1.778" layer="97"/>
+</instance>
+<instance part="TP3" gate="G$1" x="66.04" y="25.4" smashed="yes">
+<attribute name="NAME" x="64.77" y="26.67" size="1.778" layer="95"/>
+<attribute name="TP_SIGNAL_NAME" x="67.31" y="24.13" size="1.778" layer="97"/>
+</instance>
+<instance part="TP4" gate="G$1" x="66.04" y="20.32" smashed="yes">
+<attribute name="NAME" x="64.77" y="21.59" size="1.778" layer="95"/>
+<attribute name="TP_SIGNAL_NAME" x="67.31" y="19.05" size="1.778" layer="97"/>
+</instance>
+<instance part="TP5" gate="G$1" x="66.04" y="15.24" smashed="yes">
+<attribute name="NAME" x="64.77" y="16.51" size="1.778" layer="95"/>
+<attribute name="TP_SIGNAL_NAME" x="67.31" y="13.97" size="1.778" layer="97"/>
 </instance>
 </instances>
@@
 <wire x1="81.28" y1="12.7" x2="66.04" y2="12.7" width="0.1524" layer="91"/>
 <label x="68.58" y="12.7" size="1.778" layer="95"/>
+<pinref part="TP5" gate="G$1" pin="PP"/>
 </segment>
 </net>
@@
 <wire x1="81.28" y1="17.78" x2="66.04" y2="17.78" width="0.1524" layer="91"/>
 <label x="68.58" y="17.78" size="1.778" layer="95"/>
+<pinref part="TP4" gate="G$1" pin="PP"/>
 </segment>
 </net>
@@
 <wire x1="81.28" y1="22.86" x2="66.04" y2="22.86" width="0.1524" layer="91"/>
 <label x="68.58" y="22.86" size="1.778" layer="95"/>
+<pinref part="TP3" gate="G$1" pin="PP"/>
 </segment>
 </net>
@@
 <wire x1="81.28" y1="27.94" x2="66.04" y2="27.94" width="0.1524" layer="91"/>
 <label x="68.58" y="27.94" size="1.778" layer="95"/>
+<pinref part="TP2" gate="G$1" pin="PP"/>
 </segment>
 </net>
@@
 </segment>
 </net>
-<net name="INPUT2" class="0">
+<net name="INPUT2" class="1">
 <segment>
 <wire x1="180.34" y1="134.62" x2="180.34" y2="135.89" width="0.1524" layer="91"/>
